Commit message: 修改碰撞模型判断:增加仿真速度

File: resources/wheel_leg_v3/urdf/wheel_leg_v3.urdf (robot description, URDF)
Before this commit: robot wheel_leg_v3, 9 links, 8 joints
Links:
- link base_link: geometry collision box size=0.47 0.3 0.19; visual mesh filename=../meshes/base_link.STL
- link left_knee_link: geometry collision cylinder length=0.034 radius=0.0925; visual mesh filename=../meshes/left_knee_link.STL
- link left_pitch_link: geometry collision box size=0.2 0.07 0.05; visual mesh filename=../meshes/left_pitch_link.STL
- link left_roll_link: geometry visual mesh filename=../meshes/left_roll_link.STL
- link right_knee_link: geometry collision box size=0.2 0.07 0.05; visual mesh filename=../meshes/right_knee_link.STL
- link right_pitch_link: geometry visual mesh filename=../meshes/right_pitch_link.STL
- link right_roll_link: geometry visual mesh filename=../meshes/right_roll_link.STL
- link right_wheel_link: geometry collision cylinder length=0.034 radius=0.0925; visual mesh filename=../meshes/right_wheel_link.STL

Commit message: 修改轮子碰撞面积

File: resources/wheel_leg_v3/urdf/wheel_leg_v3.urdf (robot description, URDF)
Before this commit: robot wheel_leg_v3, 9 links, 8 joints
Links:
- link base_link: mass 3.010 -> 13.010
- link left_pitch_link: geometry visual mesh filename=../meshes/left_pitch_link.STL
- link left_wheel_link: geometry collision cylinder length=0.034 radius=0.0925; visual mesh filename=../meshes/left_wheel_link.STL
