Commit message: 增加resume之前训练模型的功能 修改初始位置为复位姿态 取消倒地重启 增大倒地接触乘法

File: resources/wheel_leg_v6/urdf/wheel_leg_v6.urdf (robot description, URDF)
Before this commit: robot wheel_leg_v6, 9 links, 8 joints
Links:
- link base_link: geometry collision box size=0.3 0.4 0.19; visual mesh filename=../meshes/base_link.STL

Commit message: 修改起始位置姿态 修改部分奖励

File: resources/wheel_leg_v6/urdf/wheel_leg_v6.urdf (robot description, URDF)
Before this commit: robot wheel_leg_v6, 9 links, 8 joints
Links:
- link base_link: mass 13.010 -> 3.010
- link left_leg_3: geometry collision box size=0.20 0.07 0.05; visual mesh filename=../meshes/left_leg_3.STL
- link right_leg_3: geometry collision box size=0.20 0.07 0.05; visual mesh filename=../meshes/right_leg_3.STL
Joints:
- joint joint_left_leg_2: limit lower=-1.919862 upper=3.490659 effort=45 velocity=25 -> lower=-3.14 upper=3.14 effort=45 velocity=25
- joint joint_left_leg_3: limit lower=-2.670354 upper=-0.698132 effort=45 velocity=25 -> lower=-3.14 upper=3.14 effort=45 velocity=25
- joint joint_right_leg_2: limit lower=-1.919862 upper=3.490659 effort=45 velocity=25 -> lower=-3.14 upper=3.14 effort=45 velocity=25
- joint joint_right_leg_3: limit lower=-2.670354 upper=-0.698132 effort=45 velocity=25 -> lower=-3.14 upper=3.14 effort=45 velocity=25

Commit message: flat训练效果很好 10000轮pt模型 constraint调整奖励项

File: resources/wheel_leg_v6/urdf/wheel_leg_v6.urdf (robot description, URDF)
Before this commit: robot wheel_leg_v6, 9 links, 8 joints
Joints:
- joint joint_left_leg_1: limit lower=-0.7854 upper=0.7854 effort=45 velocity=25 -> lower=-3.14 upper=3.14 effort=54 velocity=25
- joint joint_left_leg_2: limit lower=-3.14 upper=3.14 effort=45 velocity=25 -> lower=-3.14 upper=3.14 effort=14 velocity=25
- joint joint_left_leg_3: limit lower=-3.14 upper=3.14 effort=45 velocity=25 -> lower=-3.14 upper=3.14 effort=7 velocity=25
- joint joint_left_leg_4: limit lower=-999999 upper=999999 effort=15 velocity=20 -> lower=-999999 upper=999999 effort=7 velocity=20
- joint joint_right_leg_1: limit lower=-0.7854 upper=0.785398 effort=45 velocity=25 -> lower=-0.7854 upper=0.785398 effort=54 velocity=25
- joint joint_right_leg_2: limit lower=-3.14 upper=3.14 effort=45 velocity=25 -> lower=-3.14 upper=3.14 effort=14 velocity=25
- joint joint_right_leg_3: limit lower=-3.14 upper=3.14 effort=45 velocity=25 -> lower=-3.14 upper=3.14 effort=7 velocity=25
- joint joint_right_leg_4: limit lower=-999999 upper=999999 effort=15 velocity=20 -> lower=-999999 upper=999999 effort=7 velocity=20

Commit message: 调整约束范围和约束阈值

File: resources/wheel_leg_v6/urdf/wheel_leg_v6.urdf (robot description, URDF)
Before this commit: robot wheel_leg_v6, 9 links, 8 joints
Links:
- link left_leg_3: geometry collision box size=0.20 0.055 0.05; visual mesh filename=../meshes/left_leg_3.STL
- link right_leg_3: geometry collision box size=0.20 0.055 0.05; visual mesh filename=../meshes/right_leg_3.STL

Commit message: 增加力矩debug 調整constraint獎勵

File: resources/wheel_leg_v6/urdf/wheel_leg_v6.urdf (robot description, URDF)
Before this commit: robot wheel_leg_v6, 9 links, 8 joints
Joints:
- joint joint_left_leg_1: limit lower=-3.14 upper=3.14 effort=54 velocity=25 -> lower=-3.14 upper=3.14 effort=540 velocity=250
- joint joint_left_leg_2: limit lower=-3.14 upper=3.14 effort=14 velocity=25 -> lower=-3.14 upper=3.14 effort=140 velocity=250
- joint joint_left_leg_3: limit lower=-3.14 upper=3.14 effort=7 velocity=25 -> lower=-3.14 upper=3.14 effort=70 velocity=250
- joint joint_left_leg_4: limit lower=-999999 upper=999999 effort=7 velocity=20 -> lower=-999999 upper=999999 effort=70 velocity=200
- joint joint_right_leg_1: limit lower=-0.7854 upper=0.785398 effort=54 velocity=25 -> lower=-0.7854 upper=0.785398 effort=540 velocity=250
- joint joint_right_leg_2: limit lower=-3.14 upper=3.14 effort=14 velocity=25 -> lower=-3.14 upper=3.14 effort=140 velocity=250
- joint joint_right_leg_3: limit lower=-3.14 upper=3.14 effort=7 velocity=25 -> lower=-3.14 upper=3.14 effort=70 velocity=250
- joint joint_right_leg_4: limit lower=-999999 upper=999999 effort=7 velocity=20 -> lower=-999999 upper=999999 effort=70 velocity=200

Commit message: 减少cost数目 训练constraint

File: resources/wheel_leg_v6/urdf/wheel_leg_v6.urdf (robot description, URDF)
Before this commit: robot wheel_leg_v6, 9 links, 8 joints
Joints:
- joint joint_left_leg_1: limit lower=-3.14 upper=3.14 effort=540 velocity=250 -> lower=-3.14 upper=3.14 effort=54 velocity=25
- joint joint_left_leg_2: limit lower=-3.14 upper=3.14 effort=140 velocity=250 -> lower=-3.14 upper=3.14 effort=45 velocity=25
- joint joint_left_leg_3: limit lower=-3.14 upper=3.14 effort=70 velocity=250 -> lower=-3.14 upper=3.14 effort=45 velocity=25
- joint joint_left_leg_4: limit lower=-999999 upper=999999 effort=70 velocity=200 -> lower=-999999 upper=999999 effort=45 velocity=20
- joint joint_right_leg_1: limit lower=-0.7854 upper=0.785398 effort=540 velocity=250 -> lower=-0.7854 upper=0.785398 effort=54 velocity=25
- joint joint_right_leg_2: limit lower=-3.14 upper=3.14 effort=140 velocity=250 -> lower=-3.14 upper=3.14 effort=45 velocity=25
- joint joint_right_leg_3: limit lower=-3.14 upper=3.14 effort=70 velocity=250 -> lower=-3.14 upper=3.14 effort=45 velocity=25
- joint joint_right_leg_4: limit lower=-999999 upper=999999 effort=70 velocity=200 -> lower=-999999 upper=999999 effort=45 velocity=20
